Commit message: Replace teleport-grasp with real 3-DOF arm + DetachableJoint pickup
Drops the visually-meaningless "teleport bottle to tray" hack and
rebuilds v1 around a proper mobile-manipulator:

URDF (pos_v1_description/urdf/pos_robot.urdf)
- 3-DOF arm: shoulder pitch, elbow pitch, wrist pitch (axes Y).
  Link lengths 0.25 + 0.20 + 0.05 m, sized so the gripper reaches
  the shelf at world x ≈ 1.88 when the robot stops at x ≈ 1.5.
  Arm structure mirrors a Robotis OpenManipulator-X on a small
  diff-drive base — the standard ROS-tutorial mobile manipulator —
  built from scratch in URDF to avoid external pkg dependencies.
- Parallel-jaw gripper: two prismatic fingers (range 0 to 0.045 m
  per side). The joint axes mirror so the same positive command
  opens both. Sized to clear a 33 mm can radius with margin.
- gz-sim joint-position-controller plugins per actuated joint, each
  subscribing to a std_msgs/Float64 (= gz.msgs.Double) topic.
- gz-sim-detachable-joint-system plugin: gripper_base <-> soda_can.
  Starts ATTACHED at world load; the task detaches at startup so the
  can rests on the shelf, attaches at grasp time, detaches at release.

World (pos_v1_bringup/worlds/store.sdf)
- Three "bottles" replaced with a single soda_can model at the
  front edge of the shelf. Real-world 355 ml dimensions: 33 mm
  radius, 123 mm height, 0.355 kg mass, with inertia computed from
  the cylinder formula. Position chosen so the arm reaches it
  without the base colliding with the shelf.

Bridge (pos_v1_bringup/config/gz_bridge.yaml)
- Adds five std_msgs/Float64 topics for the arm + gripper joints.
- Adds two std_msgs/Empty topics for /grasp/attach and /grasp/detach.

Task (pos_v1_task/pos_v1_task/pick_and_place.py)
- 11-stage sequence: detach -> stow -> drive -> pre-grasp -> grasp ->
  close -> attach -> lift -> carry -> drive back -> place -> detach +
  open -> stow. All timing is sim-time-based.
- Hand-tuned POSE_* and GRIPPER_* constants exposed at the top of
  the file for the user to nudge if the gripper misses the can.

README
- Rewritten to document the new architecture, sequence stages, the
  PID-tuning + arm-pose-tuning knobs, and the deferred work for
  later versions (ros2_control, friction grasp, Nav2, MoveIt, etc).

Co-Authored-By: Claude Opus 4.7 (1M context) <noreply@anthropic.com>

File: v1_simple_pick/pos_v1_description/urdf/pos_robot.urdf (robot description, URDF)
Before this commit: robot pos_robot, 7 links, 6 joints
Links:
- removed link arm_segment
- added link arm_elbow, mass 0.20; collision box size=0.20 0.04 0.04; visual box size=0.20 0.04 0.04
- added link arm_shoulder, mass 0.30; collision box size=0.25 0.045 0.045; visual box size=0.25 0.045 0.045
- added link arm_wrist, mass 0.08; collision box size=0.05 0.04 0.04; visual box size=0.05 0.04 0.04
- added link gripper_base, mass 0.10; collision box size=0.05 0.06 0.04; visual box size=0.05 0.06 0.04
- added link left_finger, mass 0.02; collision box size=0.06 0.005 0.05; visual box size=0.06 0.005 0.05
- added link right_finger, mass 0.02; collision box size=0.06 0.005 0.05; visual box size=0.06 0.005 0.05
- link arm_column: mass 0.5 -> 0.6; geometry collision cylinder length=0.40 radius=0.035; visual cylinder length=0.40 radius=0.035
Joints:
- removed joint arm_segment_joint
- added joint arm_elbow_joint: type revolute, parent arm_shoulder, child arm_elbow, origin xyz=0.25 0 0 rpy=0 0 0, axis 0 1 0, limit lower=-2.5 upper=2.5 effort=20 velocity=2.0
- added joint arm_shoulder_joint: type revolute, parent arm_column, child arm_shoulder, origin xyz=0 0 0.40 rpy=0 0 0, axis 0 1 0, limit lower=-1.6 upper=1.6 effort=25 velocity=2.0
- added joint arm_wrist_joint: type revolute, parent arm_elbow, child arm_wrist, origin xyz=0.20 0 0 rpy=0 0 0, axis 0 1 0, limit lower=-2.0 upper=2.0 effort=15 velocity=2.0
- added joint gripper_base_joint: type fixed, parent arm_wrist, child gripper_base, origin xyz=0.05 0 0 rpy=0 0 0
- added joint left_finger_joint: type prismatic, parent gripper_base, child left_finger, origin xyz=0.05 0 0 rpy=0 0 0, axis 0 1 0, limit lower=0.0 upper=0.045 effort=20 velocity=0.2
- added joint right_finger_joint: type prismatic, parent gripper_base, child right_finger, origin xyz=0.05 0 0 rpy=0 0 0, axis 0 -1 0, limit lower=0.0 upper=0.045 effort=20 velocity=0.2
- joint arm_column_joint: origin xyz=-0.2 0 0.285 rpy=0 0 0 -> xyz=-0.20 0 0.075 rpy=0 0 0

Commit message: Tier 2: ros2_control + JTC, friction grasp, analytical 3-DOF IK
Replaces three Tier-1 hacks at once. The arm and gripper are now
driven by joint_trajectory_controller with PID gains in
controllers.yaml, hosted in-process by gz_ros2_control. Cartesian
arm targets are solved by a new analytical inverse-kinematics
module (ik.py). The grasp is contact-based: fingers are commanded
inward past the can's surface and the trajectory PID's saturated
effort becomes the squeeze.

URDF (pos_v1_description/urdf/pos_robot.urdf)
- File is now xacro so the gz_ros2_control plugin's <parameters>
  can use $(find pos_v1_bringup) to resolve to an absolute path.
- New <ros2_control> block with effort interfaces on the arm +
  gripper joints and state-only interfaces on the drive wheels
  (still driven by gz-sim DiffDrive; joint_state_broadcaster
  publishes their state).
- Removed: 5x gz-sim-joint-position-controller plugins, the
  DetachableJoint plugin, and gz-sim-joint-state-publisher.
- Added: high friction (mu=2.0, kp/kd contact stiffness tuning)
  on the finger pads so the gripper can actually hold the can.
- Bumped base_link mass 5->12 kg and arm_column mass 0.6->2.0 kg
  with ~5x larger inertia so the cantilevered arm can't pitch
  the base forward (root cause of the visible column tilt in
  earlier screenshots).

Controllers config (pos_v1_bringup/config/controllers.yaml — NEW)
- controller_manager @ 100 Hz
- joint_state_broadcaster
- arm_controller: joint_trajectory_controller, effort interface,
  per-joint PID gains tuned conservatively (shoulder p=250, i=20,
  d=25 etc).
- gripper_controller: same, with goal_time=0 so the controller
  doesn't report failure when the fingers can't fully close
  (i.e. when they're squeezing a can).

Bridge (pos_v1_bringup/config/gz_bridge.yaml)
- Dropped 7 topics: arm/*_cmd, gripper/*_cmd, /joint_states,
  /grasp/{attach,detach}. ros2_control handles all of these
  internally now. Only /clock, /cmd_vel and /odom still cross
  the bridge.

Launch (pos_v1_bringup/launch/sim.launch.py)
- Processes the URDF through xacro at launch time.
- Adds three controller_manager spawner Nodes chained via
  RegisterEventHandler/OnProcessExit so they fire in order
  after spawn_robot: jsb -> arm_controller -> gripper_controller.

Task script (pos_v1_task/pos_v1_task/pick_and_place.py)
- Rewritten to publish trajectory_msgs/JointTrajectory to
  /arm_controller/joint_trajectory and
  /gripper_controller/joint_trajectory instead of per-joint
  Float64.
- All pose targets are now world-frame or robot-frame Cartesian
  (CAN_X/CAN_Z, CARRY_ROBOT_XZ, PLACE_ROBOT_XZ). Joint angles
  come from ik.py.
- Friction-grasp sequence: GRIPPER_GRASP = 0.018 m (well inside
  the 33 mm can radius) so the PID saturates effort against the
  can. No /grasp/* messages anywhere.

IK module (pos_v1_task/pos_v1_task/ik.py — NEW)
- ik_solve(x, z, phi, elbow_up=True) for the planar 3-DOF arm.
- Link lengths a1=0.25, a2=0.20, a3=0.13 (last includes wrist
  link + palm + finger half-length).
- Returns (shoulder, elbow, wrist) joint angles or raises
  IKError on unreachable / singular targets.
- shoulder_frame() helper transforms world (x_w, z_w, robot_x)
  -> shoulder-frame (x, z) so the task script can specify
  Cartesian world targets directly.

Package deps
- pos_v1_bringup adds: xacro, gz_ros2_control, controller_manager,
  joint_state_broadcaster, joint_trajectory_controller.
- pos_v1_task adds: trajectory_msgs, builtin_interfaces.

README: rewritten to document the new architecture, install
requirements (apt packages for ros2_control), tunable knobs
(Cartesian targets, PID gains, friction), and the failure-mode
checklist (grasp slipping -> increase finger p / mu; arm sag
-> increase i_clamp; etc).

Untested on a Gazebo machine — the gz_ros2_control bring-up,
PID gains, and arm-pose targets will likely need 1-2 iterations
of nudging once it actually runs.

Co-Authored-By: Claude Opus 4.7 (1M context) <noreply@anthropic.com>

File: v1_simple_pick/pos_v1_description/urdf/pos_robot.urdf (robot description, URDF)
Before this commit: robot pos_robot, 12 links, 11 joints
Links:
- link arm_column: mass 0.6 -> 2.0
- link base_link: mass 5.0 -> 12.0
Joints:
- joint arm_column_joint: origin xyz=-0.20 0 0.075 rpy=0 0 0 -> xyz=-0.15 0 0.075 rpy=0 0 0
- joint arm_elbow_joint: limit lower=-2.5 upper=2.5 effort=20 velocity=2.0 -> lower=-2.5 upper=2.5 effort=30 velocity=2.0
- joint arm_shoulder_joint: limit lower=-1.6 upper=1.6 effort=25 velocity=2.0 -> lower=-1.6 upper=1.6 effort=40 velocity=2.0
- joint arm_wrist_joint: limit lower=-2.0 upper=2.0 effort=15 velocity=2.0 -> lower=-2.0 upper=2.0 effort=20 velocity=2.0
- joint left_finger_joint: limit lower=0.0 upper=0.045 effort=20 velocity=0.2 -> lower=0.005 upper=0.045 effort=40 velocity=0.2
- joint right_finger_joint: limit lower=0.0 upper=0.045 effort=20 velocity=0.2 -> lower=0.005 upper=0.045 effort=40 velocity=0.2
