Commit message: Lift base_link off the ground so the wheels actually carry the load
Previously left/right_wheel_joint had z=-0.025 in the base frame, which
put the wheel BOTTOMS at exactly the same height as base_link's bottom
(both at z=-0.075 in base frame). When the robot dropped onto the
ground, its belly contacted at the same instant the wheels did, so the
wheels carried near-zero normal force; with mu*N ~= 0 the wheels spun
without traction and the robot sat still no matter what /cmd_vel said.
That's why STAGE 1 looked like it ran (the script published cmd_vel)
but the robot didn't move, and STAGE 2 then commanded an arm pose that
was out of reach (=> the joint_trajectory_controller tolerance errors
at the joint velocity limit).

Drop the wheels and caster 5cm so the wheel bottoms protrude below the
base. Settled, base_link sits at world z=0.125 (5cm of ground
clearance) and the wheels carry the full weight. Spawn z bumped to
0.15 so the robot doesn't spawn with the wheels already in the ground,
and ik.py's SHOULDER_Z_WORLD bumped to 0.6 to match the new settled
shoulder height so the gripper still closes on the can centre.

Also added a short "What this is" section to README explaining that
v1_simple_pick is the open-loop scripted demo / mechanical baseline
(no perception, no nav) and what the real-world path on top of it
looks like.

File: v1_simple_pick/pos_v1_description/urdf/pos_robot.urdf (robot description, URDF)
Before this commit: robot pos_robot, 12 links, 11 joints
Joints:
- joint caster_joint: origin xyz=0.20 0 -0.05 rpy=0 0 0 -> xyz=0.20 0 -0.10 rpy=0 0 0
- joint left_wheel_joint: origin xyz=0 0.215 -0.025 rpy=0 0 0 -> xyz=0 0.215 -0.075 rpy=0 0 0
- joint right_wheel_joint: origin xyz=0 -0.215 -0.025 rpy=0 0 0 -> xyz=0 -0.215 -0.075 rpy=0 0 0
