Commit message: Fix spawn_robot launch crash: drop xacro pi redefinition
The xacro processor provides ${pi} as a built-in symbol. Redefining it
in robot.urdf.xacro emitted a "redefining global symbol: pi" warning on
stderr, which launch.Command treats as fatal by default — so the URDF
never reached /robot_description and the robot never spawned. Gazebo
opened the world but the launch hung before the spawn step.

Two changes:
- Remove the <xacro:property name="pi" ...> line; rely on xacro's
  built-in. All ${pi} references in the URDF keep working unchanged.
- Set Command(..., on_stderr='warn') in the launch so a future benign
  xacro warning logs instead of killing the launch.

Co-Authored-By: Claude Opus 4.7 (1M context) <noreply@anthropic.com>

File: v2/pos_v2_description/urdf/robot.urdf.xacro (robot description, xacro)
@@ -1,5 +1,5 @@
 <?xml version="1.0"?>
 <robot xmlns:xacro="http://www.ros.org/wiki/xacro" name="pos_v2_robot">
-  <xacro:property name="pi" value="3.14159265359"/>
+  <!-- ${pi} is a xacro built-in; do not redefine it (xacro warns -> launch.Command treats stderr as fatal). -->
   <!-- Base dimensions: small AGV, fits aisles and door easily. -->
   <xacro:property name="base_length" value="0.4"/>
